Commit message: Add the muscle frames in the Template

File: models/humanModelTemplate/humanModelTemplate_shoulder_Cylinder.urdf (robot description, URDF)
Before this commit: robot HumanModel, 55 links, 54 joints
Links:
- removed link MiddleTrunk
- removed link MiddleTrunk_f1
- removed link MiddleTrunk_f2
- removed link UpperTrunk_Left
- removed link UpperTrunk_Left_f1
- removed link UpperTrunk_Left_f2
- removed link UpperTrunk_Middle
- removed link UpperTrunk_Middle_f1
- removed link UpperTrunk_Middle_f2
- removed link UpperTrunk_Right
- removed link UpperTrunk_Right_f1
- removed link UpperTrunk_Right_f2
- added link BicBrac_LFA, mass 0
- added link BicBrac_LUA, mass 0
- added link BicBrac_RFA, mass 0
- added link BicBrac_RUA, mass 0
- added link BicFem_LLL, mass 0
- added link BicFem_LUL, mass 0
- added link BicFem_RLL, mass 0
- added link BicFem_RUL, mass 0
- added link ErSpin_LP, mass 0
- added link ErSpin_LUT, mass 0
- added link ErSpin_RP, mass 0
- added link ErSpin_RUT, mass 0
- added link ExtCarp_LFA, mass 0
- added link ExtCarp_LH, mass 0
- added link ExtCarp_RFA, mass 0
- added link ExtCarp_RH, mass 0
- added link FlexCarp_LFA, mass 0
- added link FlexCarp_LH, mass 0
- added link FlexCarp_RFA, mass 0
- added link FlexCarp_RH, mass 0
- added link GasLat_LF, mass 0
- added link GasLat_LUL, mass 0
- added link GasLat_RF, mass 0
- added link GasLat_RUL, mass 0
- added link GasMed_LF, mass 0
- added link GasMed_LUL, mass 0
- added link GasMed_RF, mass 0
- added link GasMed_RUL, mass 0
- added link LeftC7Shoulder_f1, mass 0
- added link LeftC7Shoulder_f2, mass 0
- added link LeftHandCOM, mass 0.00001; visual box size=0 0 0
- added link LeftShoulder, mass 6.3444; collision cylinder length=0.1 radius=0.03; visual cylinder length=0.1 radius=0.03
- added link LeftToe, mass 0.00001; visual box size=0 0 0
- added link LowerTrunk, mass 6.3444; collision box size=0.15 0.25 0.2; visual box size=0.15 0.25 0.2
- added link LowerTrunk_f1, mass 0
- added link LowerTrunk_f2, mass 0
- added link RecAbd_LP, mass 0
- added link RecAbd_LUT, mass 0
- added link RecAbd_RP, mass 0
- added link RecAbd_RUT, mass 0
- added link RecFem_LLL, mass 0
- added link RecFem_LLT, mass 0
- added link RecFem_RLL, mass 0
- added link RecFem_RLT, mass 0
- added link RightC7Shoulder_f1, mass 0
- added link RightC7Shoulder_f2, mass 0
- added link RightHandCOM, mass 0.00001; visual box size=0 0 0
- added link RightShoulder, mass 6.3444; collision cylinder length=0.1 radius=0.03; visual cylinder length=0.1 radius=0.03
- added link RightToe, mass 0.00001; visual box size=0 0 0
- added link TibAnt_LF, mass 0
- added link TibAnt_LLL, mass 0
- added link TibAnt_RF, mass 0
- added link TibAnt_RLL, mass 0
- added link TricBrac_LFA, mass 0
- added link TricBrac_LUA, mass 0
- added link TricBrac_RFA, mass 0
- added link TricBrac_RUA, mass 0
- added link UpperTrunk, mass 6.3444; collision box size=0.15 0.1 0.1; visual box size=0.15 0.1 0.1
- added link UpperTrunk_f1, mass 0
- added link UpperTrunk_f2, mass 0
Joints:
- removed joint jL4L3_rotx
- removed joint jL4L3_roty
- removed joint jL4L3_rotz
- removed joint jLeftC7Shoulder_rotx
- removed joint jLeftC7Shoulder_roty
- removed joint jLeftC7Shoulder_rotz
- removed joint jRightC7Shoulder_rotx
- removed joint jRightC7Shoulder_roty
- removed joint jRightC7Shoulder_rotz
- removed joint jT1C7_Left_rotx
- removed joint jT1C7_Left_roty
- removed joint jT1C7_Left_rotz
- removed joint jT1C7_Right_rotx
- removed joint jT1C7_Right_roty
- removed joint jT1C7_Right_rotz
- added joint jC7LeftShoulder_rotx: type revolute, parent UpperTrunk, child LeftC7Shoulder_f1, origin xyz=0   0.05    0.07 rpy=0 0 0, axis 1 0 0, limit lower=-10.0 upper=10.0 effort=30 velocity=1.0
- added joint jC7LeftShoulder_roty: type revolute, parent LeftC7Shoulder_f1, child LeftC7Shoulder_f2, origin xyz=0 0 0 rpy=0 0 0, axis 0 1 0, limit lower=-10.0 upper=10.0 effort=30 velocity=1.0
- added joint jC7LeftShoulder_rotz: type revolute, parent LeftC7Shoulder_f2, child LeftShoulder, origin xyz=0 0 0 rpy=0 0 0, axis 0 0 1, limit lower=-10.0 upper=10.0 effort=30 velocity=1.0
- added joint jC7RightShoulder_rotx: type revolute, parent UpperTrunk, child RightC7Shoulder_f1, origin xyz=0   -0.05    0.07 rpy=0 0 0, axis 1 0 0, limit lower=-10.0 upper=10.0 effort=30 velocity=1.0
- added joint jC7RightShoulder_roty: type revolute, parent RightC7Shoulder_f1, child RightC7Shoulder_f2, origin xyz=0 0 0 rpy=0 0 0, axis 0 1 0, limit lower=-10.0 upper=10.0 effort=30 velocity=1.0
- added joint jC7RightShoulder_rotz: type revolute, parent RightC7Shoulder_f2, child RightShoulder, origin xyz=0 0 0 rpy=0 0 0, axis 0 0 1, limit lower=-10.0 upper=10.0 effort=30 velocity=1.0
- added joint jLeftBallFoot_roty: type fixed, parent LeftFoot, child LeftToe, origin xyz=0.2 0 -0.05 rpy=0 0 0, axis 0 0 0
- added joint jLeftBicBrac_LFA: type fixed, parent LeftForeArm, child BicBrac_LFA, origin xyz=0.02    0   0 rpy=0 0 0, axis 0 0 0
- added joint jLeftBicBrac_LUA: type fixed, parent LeftUpperArm, child BicBrac_LUA, origin xyz=0    0   0.03 rpy=0 0 0, axis 0 0 0
- added joint jLeftErSpin_LP: type fixed, parent Pelvis, child ErSpin_LP, origin xyz=-0.075    0   0 rpy=0 0 0, axis 0 0 0
- added joint jLeftErSpin_LUT: type fixed, parent UpperTrunk, child ErSpin_LUT, origin xyz=-0.075    0.05   0.1 rpy=0 0 0, axis 0 0 0
- added joint jLeftExtCarp_LFA: type fixed, parent LeftForeArm, child ExtCarp_LFA, origin xyz=0.02   0    0 rpy=0 0 0, axis 0 0 0
- added joint jLeftExtCarp_LH: type fixed, parent LeftHand, child ExtCarp_LH, origin xyz=0.015    0.05   -0.015 rpy=0 0 0, axis 0 0 0
- added joint jLeftFlexCarp_LH: type fixed, parent LeftHand, child FlexCarp_LH, origin xyz=0.015    0.05   0.015 rpy=0 0 0, axis 0 0 0
- added joint jLeftGasLat_LF: type fixed, parent LeftFoot, child GasLat_LF, origin xyz=0    0    -0.025 rpy=0 0 0, axis 0 0 0
- added joint jLeftGasLat_LUL: type fixed, parent LeftUpperLeg, child GasLat_LUL, origin xyz=-0.0433    0.025    -0.4 rpy=0 0 0, axis 0 0 0
- added joint jLeftGasMed_LF: type fixed, parent LeftFoot, child GasMed_LF, origin xyz=0    0    -0.025 rpy=0 0 0, axis 0 0 0
- added joint jLeftGasMed_LUL: type fixed, parent LeftUpperLeg, child GasMed_LUL, origin xyz=-0.0433    -0.025    -0.4 rpy=0 0 0, axis 0 0 0
- added joint jLeftHandCOM: type fixed, parent LeftHand, child LeftHandCOM, origin xyz=0 0.05 0 rpy=0 0 0, axis 0 0 0
- added joint jLeftRecAbd_RP: type fixed, parent Pelvis, child RecAbd_LP, origin xyz=0.075    0   0 rpy=0 0 0, axis 0 0 0
- added joint jLeftRecAbd_RUT: type fixed, parent UpperTrunk, child RecAbd_LUT, origin xyz=0.075    0.05   0 rpy=0 0 0, axis 0 0 0
- added joint jLeftShoulder_rotx: type revolute, parent LeftShoulder, child LeftShoulder_f1, origin xyz=0    0.1    0 rpy=0 0 0, axis 1 0 0, limit lower=-10.0 upper=10.0 effort=30 velocity=1.0
- added joint jLeftShoulder_roty: type revolute, parent LeftShoulder_f1, child LeftShoulder_f2, origin xyz=0 0 0 rpy=0 0 0, axis 0 1 0, limit lower=-10.0 upper=10.0 effort=30 velocity=1.0
- added joint jLeftShoulder_rotz: type revolute, parent LeftShoulder_f2, child LeftUpperArm, origin xyz=0 0 0 rpy=0 0 0, axis 0 0 1, limit lower=-10.0 upper=10.0 effort=30 velocity=1.0
- added joint jLeftTibAnt_LF: type fixed, parent LeftFoot, child TibAnt_LF, origin xyz=0.1    -0.025    0 rpy=0 0 0, axis 0 0 0
- added joint jLeftTibAnt_LLL: type fixed, parent LeftLowerLeg, child TibAnt_LLL, origin xyz=0.03    0    0 rpy=0 0 0, axis 0 0 0
- added joint jLeftTricBrac_LFA: type fixed, parent LeftForeArm, child TricBrac_LFA, origin xyz=-0.02    0   0 rpy=0 0 0, axis 0 0 0
- added joint jLeftTricBrac_LUA: type fixed, parent LeftUpperArm, child TricBrac_LUA, origin xyz=-0.03    0   0 rpy=0 0 0, axis 0 0 0
- added joint jRightBallFoot_roty: type fixed, parent RightFoot, child RightToe, origin xyz=0.2 0 -0.05 rpy=0 0 0, axis 0 0 0
- added joint jRightBicBrac_RFA: type fixed, parent RightForeArm, child BicBrac_RFA, origin xyz=0.02    0   0 rpy=0 0 0, axis 0 0 0
- added joint jRightBicBrac_RUA: type fixed, parent RightUpperArm, child BicBrac_RUA, origin xyz=0    0   0.03 rpy=0 0 0, axis 0 0 0
- added joint jRightBicFem_LLL: type fixed, parent LeftLowerLeg, child BicFem_LLL, origin xyz=0    0.03    0 rpy=0 0 0, axis 0 0 0
- added joint jRightBicFem_LUL: type fixed, parent LeftUpperLeg, child BicFem_LUL, origin xyz=-0.05    0    0 rpy=0 0 0, axis 0 0 0
- added joint jRightBicFem_RLL: type fixed, parent RightLowerLeg, child BicFem_RLL, origin xyz=0    -0.03    0 rpy=0 0 0, axis 0 0 0
- added joint jRightBicFem_RUL: type fixed, parent RightUpperLeg, child BicFem_RUL, origin xyz=-0.05    0    0 rpy=0 0 0, axis 0 0 0
- added joint jRightErSpin_RP: type fixed, parent Pelvis, child ErSpin_RP, origin xyz=-0.075    0   0 rpy=0 0 0, axis 0 0 0
- added joint jRightErSpin_RUT: type fixed, parent UpperTrunk, child ErSpin_RUT, origin xyz=-0.075    -0.05   0.1 rpy=0 0 0, axis 0 0 0
- added joint jRightExtCarp_RFA: type fixed, parent RightForeArm, child ExtCarp_RFA, origin xyz=0.02   0    0 rpy=0 0 0, axis 0 0 0
- added joint jRightExtCarp_RH: type fixed, parent RightHand, child ExtCarp_RH, origin xyz=0.015    -0.05   -0.015 rpy=0 0 0, axis 0 0 0
- added joint jRightFlexCarp_LFA: type fixed, parent LeftForeArm, child FlexCarp_LFA, origin xyz=-0.02   0    0 rpy=0 0 0, axis 0 0 0
- added joint jRightFlexCarp_RFA: type fixed, parent RightForeArm, child FlexCarp_RFA, origin xyz=-0.02   0    0 rpy=0 0 0, axis 0 0 0
- added joint jRightFlexCarp_RH: type fixed, parent RightHand, child FlexCarp_RH, origin xyz=0.015    -0.05   0.015 rpy=0 0 0, axis 0 0 0
- added joint jRightGasLat_RF: type fixed, parent RightFoot, child GasLat_RF, origin xyz=0    0    -0.025 rpy=0 0 0, axis 0 0 0
- added joint jRightGasLat_RUL: type fixed, parent RightUpperLeg, child GasLat_RUL, origin xyz=-0.043    -0.025    -0.4 rpy=0 0 0, axis 0 0 0
- added joint jRightGasMed_RF: type fixed, parent RightFoot, child GasMed_RF, origin xyz=0     0    -0.025 rpy=0 0 0, axis 0 0 0
- added joint jRightGasMed_RUL: type fixed, parent RightUpperLeg, child GasMed_RUL, origin xyz=-0.0433    0.025    -0.4 rpy=0 0 0, axis 0 0 0
- added joint jRightHandCOM: type fixed, parent RightHand, child RightHandCOM, origin xyz=0 -0.05 0 rpy=0 0 0, axis 0 0 0
- added joint jRightRecAbd_RP: type fixed, parent Pelvis, child RecAbd_RP, origin xyz=0.075    0   0 rpy=0 0 0, axis 0 0 0
- added joint jRightRecAbd_RUT: type fixed, parent UpperTrunk, child RecAbd_RUT, origin xyz=0.075    -0.05   0 rpy=0 0 0, axis 0 0 0
- added joint jRightRecFem_LLL: type fixed, parent LeftLowerLeg, child RecFem_LLL, origin xyz=0.03    0    0 rpy=0 0 0, axis 0 0 0
- added joint jRightRecFem_LLT: type fixed, parent Pelvis, child RecFem_LLT, origin xyz=0.075    0.083    0.05 rpy=0 0 0, axis 0 0 0
- added joint jRightRecFem_RLL: type fixed, parent RightLowerLeg, child RecFem_RLL, origin xyz=0.03    0    0 rpy=0 0 0, axis 0 0 0
- added joint jRightRecFem_RLT: type fixed, parent Pelvis, child RecFem_RLT, origin xyz=0.075    -0.083    0.05 rpy=0 0 0, axis 0 0 0
- added joint jRightShoulder_rotx: type revolute, parent RightShoulder, child RightShoulder_f1, origin xyz=0   -0.1    0 rpy=0 0 0, axis 1 0 0, limit lower=-10.0 upper=10.0 effort=30 velocity=1.0
- added joint jRightShoulder_roty: type revolute, parent RightShoulder_f1, child RightShoulder_f2, origin xyz=0 0 0 rpy=0 0 0, axis 0 1 0, limit lower=-10.0 upper=10.0 effort=30 velocity=1.0
- added joint jRightShoulder_rotz: type revolute, parent RightShoulder_f2, child RightUpperArm, origin xyz=0 0 0 rpy=0 0 0, axis 0 0 1, limit lower=-10.0 upper=10.0 effort=30 velocity=1.0
- added joint jRightTibAnt_RF: type fixed, parent RightFoot, child TibAnt_RF, origin xyz=0.1    0.025    0 rpy=0 0 0, axis 0 0 0
- added joint jRightTibAnt_RLL: type fixed, parent RightLowerLeg, child TibAnt_RLL, origin xyz=0.03    0    0 rpy=0 0 0, axis 0 0 0
- added joint jRightTricBrac_RFA: type fixed, parent RightForeArm, child TricBrac_RFA, origin xyz=-0.02    0   0 rpy=0 0 0, axis 0 0 0
- added joint jRightTricBrac_RUA: type fixed, parent RightUpperArm, child TricBrac_RUA, origin xyz=-0.03    0   0 rpy=0 0 0, axis 0 0 0
- added joint jT9T8_rotx: type revolute, parent LowerTrunk, child UpperTrunk_f1, origin xyz=0      0    0.2 rpy=0 0 0, axis 1 0 0, limit lower=-10.0 upper=10.0 effort=30 velocity=1.0
- added joint jT9T8_roty: type revolute, parent UpperTrunk_f1, child UpperTrunk_f2, origin xyz=0 0 0 rpy=0 0 0, axis 0 1 0, limit lower=-10.0 upper=10.0 effort=30 velocity=1.0
- added joint jT9T8_rotz: type revolute, parent UpperTrunk_f2, child UpperTrunk, origin xyz=0 0 0 rpy=0 0 0, axis 0 0 1, limit lower=-10.0 upper=10.0 effort=30 velocity=1.0
- joint jL5S1_rotx: child MiddleTrunk_f1 -> LowerTrunk_f1
- joint jL5S1_roty: child MiddleTrunk_f2 -> LowerTrunk_f2; parent MiddleTrunk_f1 -> LowerTrunk_f1
- joint jL5S1_rotz: child MiddleTrunk -> LowerTrunk; parent MiddleTrunk_f2 -> LowerTrunk_f2
- joint jT1C7_rotx: parent UpperTrunk_Middle -> UpperTrunk

Commit message: Fix some muscles' nomenclature

File: models/humanModelTemplate/humanModelTemplate_shoulder_Box.urdf (robot description, URDF)
Before this commit: robot HumanModel, 103 links, 102 joints
Links:
- link LeftToe: mass 0.00001 -> 0
- link RightToe: mass 0.00001 -> 0
Joints:
- removed joint jLeftRecAbd_RP
- removed joint jLeftRecAbd_RUT
- removed joint jRightBicFem_LLL
- removed joint jRightBicFem_LUL
- removed joint jRightFlexCarp_LFA
- removed joint jRightRecFem_LLL
- removed joint jRightRecFem_LLT
- removed joint jRightRecFem_RLT
- added joint jLeftBicFem_LLL: type fixed, parent LeftLowerLeg, child BicFem_LLL, origin xyz=0    0.03    0 rpy=0 0 0, axis 0 0 0
- added joint jLeftBicFem_LUL: type fixed, parent LeftUpperLeg, child BicFem_LUL, origin xyz=-0.05    0    0 rpy=0 0 0, axis 0 0 0
- added joint jLeftFlexCarp_LFA: type fixed, parent LeftForeArm, child FlexCarp_LFA, origin xyz=-0.02   0    0 rpy=0 0 0, axis 0 0 0
- added joint jLeftRecAbd_LP: type fixed, parent Pelvis, child RecAbd_LP, origin xyz=0.075    0   0 rpy=0 0 0, axis 0 0 0
- added joint jLeftRecAbd_LUT: type fixed, parent UpperTrunk, child RecAbd_LUT, origin xyz=0.075    0.05   0 rpy=0 0 0, axis 0 0 0
- added joint jLeftRecFem_LLL: type fixed, parent LeftLowerLeg, child RecFem_LLL, origin xyz=0.03    0    0 rpy=0 0 0, axis 0 0 0
- added joint jLeftRecFem_LP: type fixed, parent Pelvis, child RecFem_LLT, origin xyz=0.075    0.083    0.05 rpy=0 0 0, axis 0 0 0
- added joint jRightRecFem_RP: type fixed, parent Pelvis, child RecFem_RLT, origin xyz=0.075    -0.083    0.05 rpy=0 0 0, axis 0 0 0
- joint jLeftBallFoot_roty: axis 0 0 0 -> 0 1 0; limit (none) -> lower=-0.174533 upper=1.5708 effort=30 velocity=1.0; type fixed -> revolute
- joint jRightBallFoot_roty: axis 0 0 0 -> 0 1 0; limit (none) -> lower=-0.174533 upper=1.5708 effort=30 velocity=1.0; type fixed -> revolute

File: models/humanModelTemplate/humanModelTemplate_shoulder_Cylinder.urdf (robot description, URDF)
Before this commit: robot HumanModel, 103 links, 102 joints
Links:
- link LeftToe: mass 0.00001 -> 0
- link RightToe: mass 0.00001 -> 0
Joints:
- removed joint jLeftRecAbd_RP
- removed joint jLeftRecAbd_RUT
- removed joint jRightBicFem_LLL
- removed joint jRightBicFem_LUL
- removed joint jRightFlexCarp_LFA
- removed joint jRightRecFem_LLL
- removed joint jRightRecFem_LLT
- removed joint jRightRecFem_RLT
- added joint jLeftBicFem_LLL: type fixed, parent LeftLowerLeg, child BicFem_LLL, origin xyz=0    0.03    0 rpy=0 0 0, axis 0 0 0
- added joint jLeftBicFem_LUL: type fixed, parent LeftUpperLeg, child BicFem_LUL, origin xyz=-0.05    0    0 rpy=0 0 0, axis 0 0 0
- added joint jLeftFlexCarp_LFA: type fixed, parent LeftForeArm, child FlexCarp_LFA, origin xyz=-0.02   0    0 rpy=0 0 0, axis 0 0 0
- added joint jLeftRecAbd_LP: type fixed, parent Pelvis, child RecAbd_LP, origin xyz=0.075    0   0 rpy=0 0 0, axis 0 0 0
- added joint jLeftRecAbd_LUT: type fixed, parent UpperTrunk, child RecAbd_LUT, origin xyz=0.075    0.05   0 rpy=0 0 0, axis 0 0 0
- added joint jLeftRecFem_LLL: type fixed, parent LeftLowerLeg, child RecFem_LLL, origin xyz=0.03    0    0 rpy=0 0 0, axis 0 0 0
- added joint jLeftRecFem_LP: type fixed, parent Pelvis, child RecFem_LLT, origin xyz=0.075    0.083    0.05 rpy=0 0 0, axis 0 0 0
- added joint jRightRecFem_RP: type fixed, parent Pelvis, child RecFem_RLT, origin xyz=0.075    -0.083    0.05 rpy=0 0 0, axis 0 0 0
- joint jLeftBallFoot_roty: axis 0 0 0 -> 0 1 0; limit (none) -> lower=-0.174533 upper=1.5708 effort=30 velocity=1.0; type fixed -> revolute
- joint jRightBallFoot_roty: axis 0 0 0 -> 0 1 0; limit (none) -> lower=-0.174533 upper=1.5708 effort=30 velocity=1.0; type fixed -> revolute
