Commit message: Fixed template

File: code/models/humanModelTemplate/humanModelTemplate.urdf (robot description, URDF)
Before this commit: robot HumanModel, 93 links, 92 joints
Links:
- link LeftFTSensor: mass 0.0 -> 1e-05
- link LeftHandCOM: mass 0.0 -> 1e-05
- link RightFTSensor: mass 0.0 -> 1e-05
- link RightHandCOM: mass 0.0 -> 1e-05

Commit message: Fixed not defining masses in the template

File: code/models/humanModelTemplate/humanModelTemplate.urdf (robot description, URDF)
Before this commit: robot HumanModel, 93 links, 92 joints
Links:
- link BicBrac_LFA: mass 0.0 -> 1e-5
- link BicBrac_LUA: mass 0.0 -> 1e-5
- link BicBrac_RFA: mass 0.0 -> 1e-5
- link BicBrac_RUA: mass 0.0 -> 1e-5
- link BicFem_LLL: mass 0.0 -> 1e-5
- link BicFem_LUL: mass 0.0 -> 1e-5
- link BicFem_RLL: mass 0.0 -> 1e-5
- link BicFem_RUL: mass 0.0 -> 1e-5
- link ErSpin_LP: mass 0.0 -> 1e-5
- link ErSpin_LUT: mass 0.0 -> 1e-5
- link ErSpin_RP: mass 0.0 -> 1e-5
- link ErSpin_RUT: mass 0.0 -> 1e-5
- link ExtCarp_LFA: mass 0.0 -> 1e-5
- link ExtCarp_LH: mass 0.0 -> 1e-5
- link ExtCarp_RFA: mass 0.0 -> 1e-5
- link ExtCarp_RH: mass 0.0 -> 1e-5
- link FlexCarp_LFA: mass 0.0 -> 1e-5
- link FlexCarp_LH: mass 0.0 -> 1e-5
- link FlexCarp_RFA: mass 0.0 -> 1e-5
- link FlexCarp_RH: mass 0.0 -> 1e-5
- link GasLat_LF: mass 0.0 -> 1e-5
- link GasLat_LUL: mass 0.0 -> 1e-5
- link GasLat_RF: mass 0.0 -> 1e-5
- link GasLat_RUL: mass 0.0 -> 1e-5
- link GasMed_LF: mass 0.0 -> 1e-5
- link GasMed_LUL: mass 0.0 -> 1e-5
- link GasMed_RF: mass 0.0 -> 1e-5
- link GasMed_RUL: mass 0.0 -> 1e-5
- link Head: mass 0.0 -> 1e-5
- link Head_f1: mass 0.0 -> 1e-5
- link LeftFoot: mass 0.0 -> 1e-5
- link LeftFoot_f1: mass 0.0 -> 1e-5
- link LeftFoot_f2: mass 0.0 -> 1e-5
- link LeftForeArm: mass 0.0 -> 1e-5
- link LeftForeArm_f1: mass 0.0 -> 1e-5
- link LeftHand: mass 0.0 -> 1e-5
- link LeftHand_f1: mass 0.0 -> 1e-5
- link LeftLowerLeg: mass 0.0 -> 1e-5
- link LeftLowerLeg_f1: mass 0.0 -> 1e-5
- link LeftShoulder: mass 0.0 -> 1e-5
- link LeftShoulder_f1: mass 0.0 -> 1e-5
- link LeftShoulder_f2: mass 0.0 -> 1e-5
- link LeftToe: mass 0.0 -> 1e-5
- link LeftUpperArm: mass 0.0 -> 1e-5
- link LeftUpperLeg: mass 0.0 -> 1e-5
- link LeftUpperLeg_f1: mass 0.0 -> 1e-5
- link LeftUpperLeg_f2: mass 0.0 -> 1e-5
- link LowerTrunk: mass 0.0 -> 1e-5
- link LowerTrunk_f1: mass 0.0 -> 1e-5
- link Neck: mass 0.0 -> 1e-5
- link Neck_f1: mass 0.0 -> 1e-5
- link Neck_f2: mass 0.0 -> 1e-5
- link Pelvis: mass 0.0 -> 1e-5
- link RecAbd_LP: mass 0.0 -> 1e-5
- link RecAbd_LUT: mass 0.0 -> 1e-5
- link RecAbd_RP: mass 0.0 -> 1e-5
- link RecAbd_RUT: mass 0.0 -> 1e-5
- link RecFem_LLL: mass 0.0 -> 1e-5
- link RecFem_LLT: mass 0.0 -> 1e-5
- link RecFem_RLL: mass 0.0 -> 1e-5
- link RecFem_RLT: mass 0.0 -> 1e-5
- link RightFoot: mass 0.0 -> 1e-5
- link RightFoot_f1: mass 0.0 -> 1e-5
- link RightFoot_f2: mass 0.0 -> 1e-5
- link RightForeArm: mass 0.0 -> 1e-5
- link RightForeArm_f1: mass 0.0 -> 1e-5
- link RightHand: mass 0.0 -> 1e-5
- link RightHand_f1: mass 0.0 -> 1e-5
- link RightLowerLeg: mass 0.0 -> 1e-5
- link RightLowerLeg_f1: mass 0.0 -> 1e-5
- link RightShoulder: mass 0.0 -> 1e-5
- link RightShoulder_f1: mass 0.0 -> 1e-5
- link RightShoulder_f2: mass 0.0 -> 1e-5
- link RightToe: mass 0.0 -> 1e-5
- link RightUpperArm: mass 0.0 -> 1e-5
- link RightUpperLeg: mass 0.0 -> 1e-5
- link RightUpperLeg_f1: mass 0.0 -> 1e-5
- link RightUpperLeg_f2: mass 0.0 -> 1e-5
- link TibAnt_LF: mass 0.0 -> 1e-5
- link TibAnt_LLL: mass 0.0 -> 1e-5
- link TibAnt_RF: mass 0.0 -> 1e-5
- link TibAnt_RLL: mass 0.0 -> 1e-5
- link TricBrac_LFA: mass 0.0 -> 1e-5
- link TricBrac_LUA: mass 0.0 -> 1e-5
- link TricBrac_RFA: mass 0.0 -> 1e-5
- link TricBrac_RUA: mass 0.0 -> 1e-5
- link UpperTrunk: mass 0.0 -> 1e-5
- link UpperTrunk_f1: mass 0.0 -> 1e-5
- link UpperTrunk_f2: mass 0.0 -> 1e-5

Commit message: Corrected muscles masses

File: code/models/humanModelTemplate/humanModelTemplate.urdf (robot description, URDF)
Before this commit: robot HumanModel, 93 links, 92 joints
Links:
- link BicBrac_LFA: mass 1e-5 -> 0.0
- link BicBrac_LUA: mass 1e-5 -> 0.0
- link BicBrac_RFA: mass 1e-5 -> 0.0
- link BicBrac_RUA: mass 1e-5 -> 0.0
- link BicFem_LLL: mass 1e-5 -> 0.0
- link BicFem_LUL: mass 1e-5 -> 0.0
- link BicFem_RLL: mass 1e-5 -> 0.0
- link BicFem_RUL: mass 1e-5 -> 0.0
- link ErSpin_LP: mass 1e-5 -> 0.0
- link ErSpin_LUT: mass 1e-5 -> 0.0
- link ErSpin_RP: mass 1e-5 -> 0.0
- link ErSpin_RUT: mass 1e-5 -> 0.0
- link ExtCarp_LFA: mass 1e-5 -> 0.0
- link ExtCarp_LH: mass 1e-5 -> 0.0
- link ExtCarp_RFA: mass 1e-5 -> 0.0
- link ExtCarp_RH: mass 1e-5 -> 0.0
- link FlexCarp_LFA: mass 1e-5 -> 0.0
- link FlexCarp_LH: mass 1e-5 -> 0.0
- link FlexCarp_RFA: mass 1e-5 -> 0.0
- link FlexCarp_RH: mass 1e-5 -> 0.0
- link GasLat_LF: mass 1e-5 -> 0.0
- link GasLat_LUL: mass 1e-5 -> 0.0
- link GasLat_RF: mass 1e-5 -> 0.0
- link GasLat_RUL: mass 1e-5 -> 0.0
- link GasMed_LF: mass 1e-5 -> 0.0
- link GasMed_LUL: mass 1e-5 -> 0.0
- link GasMed_RF: mass 1e-5 -> 0.0
- link GasMed_RUL: mass 1e-5 -> 0.0
- link RecAbd_LP: mass 1e-5 -> 0.0
- link RecAbd_LUT: mass 1e-5 -> 0.0
- link RecAbd_RP: mass 1e-5 -> 0.0
- link RecAbd_RUT: mass 1e-5 -> 0.0
- link RecFem_LLL: mass 1e-5 -> 0.0
- link RecFem_LLT: mass 1e-5 -> 0.0
- link RecFem_RLL: mass 1e-5 -> 0.0
- link RecFem_RLT: mass 1e-5 -> 0.0
- link TibAnt_LF: mass 1e-5 -> 0.0
- link TibAnt_LLL: mass 1e-5 -> 0.0
- link TibAnt_RF: mass 1e-5 -> 0.0
- link TibAnt_RLL: mass 1e-5 -> 0.0
- link TricBrac_LFA: mass 1e-5 -> 0.0
- link TricBrac_LUA: mass 1e-5 -> 0.0
- link TricBrac_RFA: mass 1e-5 -> 0.0
- link TricBrac_RUA: mass 1e-5 -> 0.0

Commit message: Fixed upper arms joint limits in the template

File: code/models/humanModelTemplate/humanModelTemplate.urdf (robot description, URDF)
Before this commit: robot HumanModel, 93 links, 92 joints
Joints:
- joint jLeftShoulder_rotx: limit lower=-0.8727 upper=0.8727 effort=30 velocity=1.0 -> lower=-1.5708 upper=2.35619 effort=30 velocity=1.0
- joint jLeftShoulder_roty: limit lower=-0.8727 upper=0.8727 effort=30 velocity=1.0 -> lower=-1.5708 upper=1.5708 effort=30 velocity=1.0
- joint jLeftShoulder_rotz: limit lower=-0.8727 upper=0.8727 effort=30 velocity=1.0 -> lower=-3.14159 upper=0.785398 effort=30 velocity=1.0
- joint jRightShoulder_rotx: limit lower=-0.8727 upper=0.8727 effort=30 velocity=1.0 -> lower=-2.35619 upper=1.5708 effort=30 velocity=1.0
- joint jRightShoulder_roty: limit lower=-0.8727 upper=0.8727 effort=30 velocity=1.0 -> lower=-1.5708 upper=1.5708 effort=30 velocity=1.0
- joint jRightShoulder_rotz: limit lower=-0.8727 upper=0.8727 effort=30 velocity=1.0 -> lower=-0.785398 upper=3.14159 effort=30 velocity=1.0

Commit message: Code changes for new spinal cord model

File: code/models/humanModelTemplate/humanModelTemplate.urdf (robot description, URDF)
Before this commit: robot HumanModel, 93 links, 92 joints
Links:
- removed link LowerTrunk
- removed link LowerTrunk_f1
- removed link UpperTrunk
- removed link UpperTrunk_f1
- removed link UpperTrunk_f2
- added link C7Left_f1, mass 1e-5
- added link C7Left_f2, mass 1e-5
- added link C7Right_f1, mass 1e-5
- added link C7Right_f2, mass 1e-5
- added link L3, mass 1e-5; collision box size=1 1 1; visual box size=1 1 1
- added link L3_f1, mass 1e-5
- added link L5, mass 1e-5; collision box size=1 1 1; visual box size=1 1 1
- added link L5_f1, mass 1e-5
- added link LeftHeel, mass 1e-5; collision box size=1 1 1; visual box size=1 1 1
- added link RightHeel, mass 1e-5; collision box size=1 1 1; visual box size=1 1 1
- added link T12, mass 1e-5; collision box size=1 1 1; visual box size=1 1 1
- added link T12_f1, mass 1e-5
- added link T8, mass 1e-5; collision box size=1 1 1; visual box size=1 1 1
- added link T8_f1, mass 1e-5
- added link T8_f2, mass 1e-5
Joints:
- added joint jC7LeftShoulder_roty: type revolute, parent C7Left_f1, child C7Left_f2, origin xyz=0 0 0 rpy=0 0 0, axis 0 1 0, limit lower=-0.349066 upper=0.349066 effort=30 velocity=1.0
- added joint jC7LeftShoulder_rotz: type revolute, parent C7Left_f2, child LeftShoulder, origin xyz=0 0 0 rpy=0 0 0, axis 0 0 1, limit lower=-0.349066 upper=0.349066 effort=30 velocity=1.0
- added joint jC7RightShoulder_roty: type revolute, parent C7Right_f1, child C7Right_f2, origin xyz=0 0 0 rpy=0 0 0, axis 0 1 0, limit lower=-0.349066 upper=0.349066 effort=30 velocity=1.0
- added joint jC7RightShoulder_rotz: type revolute, parent C7Right_f2, child RightShoulder, origin xyz=0 0 0 rpy=0 0 0, axis 0 0 1, limit lower=-0.349066 upper=0.349066 effort=30 velocity=1.0
- added joint jL1T12_rotx: type revolute, parent L3, child T12_f1, origin xyz=0 0 0 rpy=0 0 0, axis 1 0 0, limit lower=-0.610865 upper=0.610865 effort=30 velocity=1.0
- added joint jL1T12_roty: type revolute, parent T12_f1, child T12, origin xyz=0 0 0 rpy=0 0 0, axis 0 1 0, limit lower=-0.523599 upper=1.309 effort=30 velocity=1.0
- added joint jL4L3_rotx: type revolute, parent L5, child L3_f1, origin xyz=0 0 0 rpy=0 0 0, axis 1 0 0, limit lower=-0.610865 upper=0.610865 effort=30 velocity=1.0
- added joint jL4L3_roty: type revolute, parent L3_f1, child L3, origin xyz=0 0 0 rpy=0 0 0, axis 0 1 0, limit lower=-0.523599 upper=1.309 effort=30 velocity=1.0
- added joint jLeftHeel_roty: type revolute, parent LeftFoot, child LeftHeel, origin xyz=0 0 0 rpy=0 0 0, axis 0 1 0, limit lower=-1.5708 upper=0.174533 effort=30 velocity=1.0
- added joint jRightHeel_roty: type revolute, parent RightFoot, child RightHeel, origin xyz=0 0 0 rpy=0 0 0, axis 0 1 0, limit lower=-1.5708 upper=0.174533 effort=30 velocity=1.0
- joint jC7LeftShoulder_rotx: child LeftShoulder -> C7Left_f1; parent UpperTrunk -> T8
- joint jC7RightShoulder_rotx: child RightShoulder -> C7Right_f1; parent UpperTrunk -> T8
- joint jL5S1_rotx: child LowerTrunk_f1 -> L5_f1
- joint jL5S1_roty: child LowerTrunk -> L5; parent LowerTrunk_f1 -> L5_f1
- joint jLeftErSpin_LUT: parent UpperTrunk -> T8
- joint jLeftRecAbd_LUT: parent UpperTrunk -> T8
- joint jRightErSpin_RUT: parent UpperTrunk -> T8
- joint jRightRecAbd_RUT: parent UpperTrunk -> T8
- joint jT1C7_rotx: parent UpperTrunk -> T8
- joint jT9T8_rotx: child UpperTrunk_f1 -> T8_f1; parent LowerTrunk -> T12
- joint jT9T8_roty: child UpperTrunk_f2 -> T8_f2; parent UpperTrunk_f1 -> T8_f1
- joint jT9T8_rotz: child UpperTrunk -> T8; parent UpperTrunk_f2 -> T8_f2

Commit message: Started adding fingers - TODO: adjust thumb

File: code/models/humanModelTemplate/humanModelTemplate.urdf (robot description, URDF)
Before this commit: robot HumanModel, 103 links, 102 joints
Links:
- added link l_hand_index_1, mass 1e-5; collision box size=1 1 1; visual box size=1 1 1
- added link l_hand_index_2, mass 1e-5; collision box size=1 1 1; visual box size=1 1 1
- added link l_hand_index_3, mass 1e-5; collision box size=1 1 1; visual box size=1 1 1
- added link l_hand_middle_1, mass 1e-5; collision box size=1 1 1; visual box size=1 1 1
- added link l_hand_middle_2, mass 1e-5; collision box size=1 1 1; visual box size=1 1 1
- added link l_hand_pinkie_1, mass 1e-5; collision box size=1 1 1; visual box size=1 1 1
- added link l_hand_pinkie_2, mass 1e-5; collision box size=1 1 1; visual box size=1 1 1
- added link l_hand_ring_1, mass 1e-5; collision box size=1 1 1; visual box size=1 1 1
- added link l_hand_ring_2, mass 1e-5; collision box size=1 1 1; visual box size=1 1 1
- added link l_hand_thumb_1, mass 1e-5; collision box size=1 1 1; visual box size=1 1 1
- added link l_hand_thumb_2, mass 1e-5; collision box size=1 1 1; visual box size=1 1 1
- added link l_hand_thumb_3, mass 1e-5; collision box size=1 1 1; visual box size=1 1 1
- added link r_hand_index_1, mass 1e-5; collision box size=1 1 1; visual box size=1 1 1
- added link r_hand_index_2, mass 1e-5; collision box size=1 1 1; visual box size=1 1 1
- added link r_hand_index_3, mass 1e-5; collision box size=1 1 1; visual box size=1 1 1
- added link r_hand_middle_1, mass 1e-5; collision box size=1 1 1; visual box size=1 1 1
- added link r_hand_middle_2, mass 1e-5; collision box size=1 1 1; visual box size=1 1 1
- added link r_hand_pinkie_1, mass 1e-5; collision box size=1 1 1; visual box size=1 1 1
- added link r_hand_pinkie_2, mass 1e-5; collision box size=1 1 1; visual box size=1 1 1
- added link r_hand_ring_1, mass 1e-5; collision box size=1 1 1; visual box size=1 1 1
- added link r_hand_ring_2, mass 1e-5; collision box size=1 1 1; visual box size=1 1 1
- added link r_hand_thumb_1, mass 1e-5; collision box size=1 1 1; visual box size=1 1 1
- added link r_hand_thumb_2, mass 1e-5; collision box size=1 1 1; visual box size=1 1 1
- added link r_hand_thumb_3, mass 1e-5; collision box size=1 1 1; visual box size=1 1 1
Joints:
- added joint l_index_add: type revolute, parent LeftHand, child l_hand_index_1, origin xyz=0.022499999999999958 -0.0015000000000005842 -0.06859999999999963 rpy=0 0 0, axis 0 0 1, limit lower=0 upper=0.2617993877991494 effort=30 velocity=1.0
- added joint l_index_dist: type revolute, parent l_hand_index_2, child l_hand_index_3, origin xyz=2.7755575615628914e-17 -0.0015000000000000568 -0.039999999999999925 rpy=0 0 0, axis 1 0 0, limit lower=0 upper=1.7165313193364231 effort=30 velocity=1.0
- added joint l_index_prox: type revolute, parent l_hand_index_1, child l_hand_index_2, origin xyz=0.009192533317427629 1.3877787807814457e-16 -0.030713451316238316 rpy=0 0 0, axis 1 0 0, limit lower=0.10035643198967395 upper=1.710422666954443 effort=30 velocity=1.0
- added joint l_middle_dist: type revolute, parent l_hand_middle_1, child l_hand_middle_2, origin xyz=-3.122502256758253e-17 -0.0015000000000000568 -0.040000000000000036 rpy=0 0 0, axis 1 0 0, limit lower=0 upper=1.7165313193364231 effort=30 velocity=1.0
- added joint l_middle_prox: type revolute, parent LeftHand, child l_hand_middle_1, origin xyz=0.009599999999999831 -0.0015000000000003344 -0.10299999999999979 rpy=0 0 0, axis 1 0 0, limit lower=0.10035643198967395 upper=1.710422666954443 effort=30 velocity=1.0
- added joint l_pinkie_dist: type revolute, parent l_hand_pinkie_1, child l_hand_pinkie_2, origin xyz=3.469446951953614e-18 -0.0014999999959518229 -0.03500000000409326 rpy=0 0 0, axis 1 0 0, limit lower=0.04852015320544236 upper=1.7763961126798287 effort=30 velocity=1.0
- added joint l_pinkie_prox: type revolute, parent LeftHand, child l_hand_pinkie_1, origin xyz=-0.035982322249527375 -0.0023883158589563247 -0.09206560929209864 rpy=0 0 0, axis 1 0 0, limit lower=0.10035643198967395 upper=1.710422666954443 effort=30 velocity=1.0
- added joint l_ring_dist: type revolute, parent l_hand_ring_1, child l_hand_ring_2, origin xyz=4.336808689942018e-18 -0.0015000000000000568 -0.03999999999999998 rpy=0 0 0, axis 1 0 0, limit lower=0 upper=1.7165313193364231 effort=30 velocity=1.0
- added joint l_ring_prox: type revolute, parent LeftHand, child l_hand_ring_1, origin xyz=-0.015417755558120076 -0.0018498137284708727 -0.09788067183884427 rpy=0 0 0, axis 1 0 0, limit lower=0.10035643198967395 upper=1.710422666954443 effort=30 velocity=1.0
- added joint l_thumb_add: type revolute, parent LeftHand, child l_hand_thumb_1, origin xyz=0.023374863256390876 -0.003000000000000086 -0.03452383847355481 rpy=0 0 0.75, axis 0 0 -1, limit lower=0 upper=1.7453292519943295 effort=30 velocity=1.0
- added joint l_thumb_dist: type revolute, parent l_hand_thumb_2, child l_hand_thumb_3, origin xyz=-2.7755575615628914e-17 -0.0037106254246525305 -0.03483505790088372 rpy=0 0 0, axis 1 0 0, limit lower=0 upper=1.7763961126798287 effort=30 velocity=1.0
- added joint l_thumb_prox: type revolute, parent l_hand_thumb_1, child l_hand_thumb_2, origin xyz=-0.03809319745034625 -0.003259193858544507 -0.0036017448037204414 rpy=0 0 0, axis 1 0 0, limit lower=0.06335545184739416 upper=1.710422666954443 effort=30 velocity=1.0
- added joint r_index_add: type revolute, parent RightHand, child r_hand_index_1, origin xyz=0.022499999999999756 0.0015000000000003344 -0.06859999999999983 rpy=0 0 0, axis 0 0 1, limit lower=0 upper=0.2617993877991494 effort=30 velocity=1.0
- added joint r_index_dist: type revolute, parent r_hand_index_2, child r_hand_index_3, origin xyz=4.440892098500626e-16 -0.0014999999999996683 -0.039999999999999925 rpy=0 0 0, axis 1 0 0, limit lower=0 upper=1.7165313193364231 effort=30 velocity=1.0
- added joint r_index_prox: type revolute, parent r_hand_index_1, child r_hand_index_2, origin xyz=-0.00919253331742792 -1.1102230246251565e-16 -0.030713451316238427 rpy=0 0 0, axis 1 0 0, limit lower=0.10035643198967395 upper=1.710422666954443 effort=30 velocity=1.0
- added joint r_middle_dist: type revolute, parent r_hand_middle_1, child r_hand_middle_2, origin xyz=3.469446951953614e-16 -0.0014999999953827503 -0.04000000000017301 rpy=0 0 0, axis 1 0 0, limit lower=0 upper=1.7165313193364231 effort=30 velocity=1.0
- added joint r_middle_prox: type revolute, parent RightHand, child r_hand_middle_1, origin xyz=0.009600000000000192 0.0015000000000006675 -0.1029999999999997 rpy=0 0 0, axis 1 0 0, limit lower=0.10035643198967395 upper=1.710422666954443 effort=30 velocity=1.0
- added joint r_pinkie_dist: type revolute, parent r_hand_pinkie_1, child r_hand_pinkie_2, origin xyz=2.8102520310824275e-16 -0.0015141933068321678 -0.03499938883222847 rpy=0 0 0, axis 1 0 0, limit lower=0.04852015320544236 upper=1.7763961126798287 effort=30 velocity=1.0
- added joint r_pinkie_prox: type revolute, parent RightHand, child r_hand_pinkie_1, origin xyz=-0.03598268094316618 0.0023777595791096284 -0.0920682813194636 rpy=0 0 0, axis 1 0 0, limit lower=0.10035643198967395 upper=1.710422666954443 effort=30 velocity=1.0
- added joint r_ring_dist: type revolute, parent r_hand_ring_1, child r_hand_ring_2, origin xyz=2.8275992658421956e-16 -0.0014999999970887745 -0.04000000000010917 rpy=0 0 0, axis 1 0 0, limit lower=0 upper=1.7165313193364231 effort=30 velocity=1.0
- added joint r_ring_prox: type revolute, parent RightHand, child r_hand_ring_1, origin xyz=-0.01541775555811984 0.0018498137284709282 -0.09788067183884414 rpy=0 0 0, axis 1 0 0, limit lower=0.10035643198967395 upper=1.710422666954443 effort=30 velocity=1.0
- added joint r_thumb_add: type revolute, parent RightHand, child r_hand_thumb_1, origin xyz=0.02337486325639067 0.0030000000000002802 -0.034523838473554336 rpy=0 0 -0.75, axis 0 0 1, limit lower=0 upper=1.7453292519943295 effort=30 velocity=1.0
- added joint r_thumb_dist: type revolute, parent r_hand_thumb_2, child r_hand_thumb_3, origin xyz=-8.326672684688674e-17 -0.0037106255282955414 -0.03483505788984376 rpy=0 0 0, axis 1 0 0, limit lower=0 upper=1.7763961126798287 effort=30 velocity=1.0
- added joint r_thumb_prox: type revolute, parent r_hand_thumb_1, child r_hand_thumb_2, origin xyz=0.03807465449956041 0.0034691095803252303 -0.003601744803549689 rpy=0 0 0, axis 1 0 0, limit lower=0.06335545184739416 upper=1.710422666954443 effort=30 velocity=1.0

Commit message: Corrected right thumb

File: code/models/humanModelTemplate/humanModelTemplate.urdf (robot description, URDF)
Before this commit: robot HumanModel, 127 links, 126 joints
Joints:
- joint r_thumb_add: axis 0 0 1 -> 1 0 0; origin xyz=0.02337486325639067 0.0030000000000002802 -0.034523838473554336 rpy=0 0 -0.75 -> xyz=0.02337486325639067 0.0030000000000002802 -0.034523838473554336 rpy=0.0 0.0 1.4
- joint r_thumb_prox: axis 1 0 0 -> 0 0 1; limit lower=0.06335545184739416 upper=1.710422666954443 effort=30 velocity=1.0 -> lower=-1.43117 upper=0.0 effort=30 velocity=1.0

Commit message: Corrected left thumb joints

File: code/models/humanModelTemplate/humanModelTemplate.urdf (robot description, URDF)
Before this commit: robot HumanModel, 127 links, 126 joints
Joints:
- joint l_thumb_add: axis 0 0 -1 -> -1 0 0; origin xyz=0.023374863256390876 -0.003000000000000086 -0.03452383847355481 rpy=0 0 0.75 -> xyz=0.023374863256390876 -0.003000000000000086 -0.03452383847355481 rpy=0 0 -1.4
- joint l_thumb_dist: limit lower=0 upper=1.7763961126798287 effort=30 velocity=1.0 -> lower=-1.7763961126798287 upper=0 effort=30 velocity=1.0
- joint l_thumb_prox: axis 1 0 0 -> 0 0 1; limit lower=0.06335545184739416 upper=1.710422666954443 effort=30 velocity=1.0 -> lower=0.0 upper=1.43117 effort=30 velocity=1.0

Commit message: Corrected joints in left hand

File: code/models/humanModelTemplate/humanModelTemplate.urdf (robot description, URDF)
Before this commit: robot HumanModel, 127 links, 126 joints
Joints:
- joint l_index_add: limit lower=0 upper=0.2617993877991494 effort=30 velocity=1.0 -> lower=-0.2617993877991494 upper=0 effort=30 velocity=1.0
- joint l_index_dist: axis 1 0 0 -> -1 0 0
- joint l_index_prox: axis 1 0 0 -> -1 0 0
- joint l_middle_dist: axis 1 0 0 -> -1 0 0
- joint l_middle_prox: axis 1 0 0 -> -1 0 0
- joint l_pinkie_dist: axis 1 0 0 -> -1 0 0
- joint l_pinkie_prox: axis 1 0 0 -> -1 0 0
- joint l_ring_dist: axis 1 0 0 -> -1 0 0
- joint l_ring_prox: axis 1 0 0 -> -1 0 0
