Commit message: Middle, ring and pinkie fingers modified into 3 links (add, prox,dist)

File: code/models/humanModelTemplate/humanModelTemplate.urdf (robot description, URDF)
Before this commit: robot HumanModel, 127 links, 126 joints
Links:
- added link l_hand_middle_3, mass 1e-5; collision box size=1 1 1; visual box size=1 1 1
- added link l_hand_pinkie_3, mass 1e-5; collision box size=1 1 1; visual box size=1 1 1
- added link l_hand_ring_3, mass 1e-5; collision box size=1 1 1; visual box size=1 1 1
- added link r_hand_middle_3, mass 1e-5; collision box size=1 1 1; visual box size=1 1 1
- added link r_hand_pinkie_3, mass 1e-5; collision box size=1 1 1; visual box size=1 1 1
- added link r_hand_ring_3, mass 1e-5; collision box size=1 1 1; visual box size=1 1 1
Joints:
- added joint l_middle_add: type revolute, parent LeftHand, child l_hand_middle_1, origin xyz=0.009599999999999831 -0.0015000000000003344 -0.10299999999999979 rpy=0 0 0, axis 0 0 1, limit lower=-0.2617993877991494 upper=0 effort=30 velocity=1.0
- added joint l_pinkie_add: type revolute, parent LeftHand, child l_hand_pinkie_1, origin xyz=-0.035982322249527375 -0.0023883158589563247 -0.09206560929209864 rpy=0 0 0, axis 0 0 1, limit lower=-0.2617993877991494 upper=0 effort=30 velocity=1.0
- added joint l_ring_add: type revolute, parent LeftHand, child l_hand_ring_1, origin xyz=-0.015417755558120076 -0.0018498137284708727 -0.09788067183884427 rpy=0 0 0, axis 0 0 1, limit lower=-0.2617993877991494 upper=0 effort=30 velocity=1.0
- added joint r_middle_add: type revolute, parent RightHand, child r_hand_middle_1, origin xyz=0.009600000000000192 0.0015000000000006675 -0.1029999999999997 rpy=0 0 0, axis 0 0 1, limit lower=0 upper=0.2617993877991494 effort=30 velocity=1.0
- added joint r_pinkie_add: type revolute, parent RightHand, child r_hand_pinkie_1, origin xyz=-0.03598268094316618 0.0023777595791096284 -0.0920682813194636 rpy=0 0 0, axis 0 0 1, limit lower=0 upper=0.2617993877991494 effort=30 velocity=1.0
- added joint r_ring_add: type revolute, parent RightHand, child r_hand_ring_1, origin xyz=-0.01541775555811984 0.0018498137284709282 -0.09788067183884414 rpy=0 0 0, axis 0 0 1, limit lower=0 upper=0.2617993877991494 effort=30 velocity=1.0
- joint l_middle_dist: child l_hand_middle_2 -> l_hand_middle_3; parent l_hand_middle_1 -> l_hand_middle_2
- joint l_middle_prox: child l_hand_middle_1 -> l_hand_middle_2; parent LeftHand -> l_hand_middle_1
- joint l_pinkie_dist: child l_hand_pinkie_2 -> l_hand_pinkie_3; parent l_hand_pinkie_1 -> l_hand_pinkie_2
- joint l_pinkie_prox: child l_hand_pinkie_1 -> l_hand_pinkie_2; parent LeftHand -> l_hand_pinkie_1
- joint l_ring_dist: child l_hand_ring_2 -> l_hand_ring_3; parent l_hand_ring_1 -> l_hand_ring_2
- joint l_ring_prox: child l_hand_ring_1 -> l_hand_ring_2; parent LeftHand -> l_hand_ring_1
- joint r_middle_dist: child r_hand_middle_2 -> r_hand_middle_3; parent r_hand_middle_1 -> r_hand_middle_2
- joint r_middle_prox: child r_hand_middle_1 -> r_hand_middle_2; parent RightHand -> r_hand_middle_1
- joint r_pinkie_dist: child r_hand_pinkie_2 -> r_hand_pinkie_3; parent r_hand_pinkie_1 -> r_hand_pinkie_2
- joint r_pinkie_prox: child r_hand_pinkie_1 -> r_hand_pinkie_2; parent RightHand -> r_hand_pinkie_1
- joint r_ring_dist: child r_hand_ring_2 -> r_hand_ring_3; parent r_hand_ring_1 -> r_hand_ring_2
- joint r_ring_prox: child r_hand_ring_1 -> r_hand_ring_2; parent RightHand -> r_hand_ring_1

Commit message: Updated lower limit fingers add

File: code/models/humanModelTemplate/humanModelTemplate.urdf (robot description, URDF)
Before this commit: robot HumanModel, 133 links, 132 joints
Joints:
- joint l_index_add: limit lower=-0.2617993877991494 upper=0 effort=30 velocity=1.0 -> lower=-0.2617993877991494 upper=0.2617993877991494 effort=30 velocity=1.0
- joint l_middle_add: limit lower=-0.2617993877991494 upper=0 effort=30 velocity=1.0 -> lower=-0.2617993877991494 upper=0.2617993877991494 effort=30 velocity=1.0
- joint l_pinkie_add: limit lower=-0.2617993877991494 upper=0 effort=30 velocity=1.0 -> lower=-0.2617993877991494 upper=0.2617993877991494 effort=30 velocity=1.0
- joint l_ring_add: limit lower=-0.2617993877991494 upper=0 effort=30 velocity=1.0 -> lower=-0.2617993877991494 upper=0.2617993877991494 effort=30 velocity=1.0
- joint r_index_add: limit lower=0 upper=0.2617993877991494 effort=30 velocity=1.0 -> lower=-0.2617993877991494 upper=0.2617993877991494 effort=30 velocity=1.0
- joint r_middle_add: limit lower=0 upper=0.2617993877991494 effort=30 velocity=1.0 -> lower=-0.2617993877991494 upper=0.2617993877991494 effort=30 velocity=1.0
- joint r_pinkie_add: limit lower=0 upper=0.2617993877991494 effort=30 velocity=1.0 -> lower=-0.2617993877991494 upper=0.2617993877991494 effort=30 velocity=1.0
- joint r_ring_add: limit lower=0 upper=0.2617993877991494 effort=30 velocity=1.0 -> lower=-0.2617993877991494 upper=0.2617993877991494 effort=30 velocity=1.0
