Commit message: Add fingers to human model (#27)
* Started adding fingers - TODO: adjust thumb

* Corrected direction left thumb

* Reduced length of pinkies

* Changed dimensions  of  thumb links

* Corrected right thumb

* Corrected left thumb joints

* Adjusted width and position of fingers

* Corrected joints in left hand

* Middle, ring and pinkie fingers modified into 3 links (add, prox,dist)

* Updated lower limit fingers add

* Added meshes for fingers

* Corrected new right hand

* Added linkdimensions and norms for adding fingers meshes

* Updated README: updated description of the URDF model

* Updated README

* Corrected number of meshes

* Replace human model overview image 

Updated image link for the human model overview in README.

* Added script and README for converting URDF to include fingers

File: code/models/humanModelTemplate/humanModelTemplate.urdf (robot description, URDF)
Before this commit: robot HumanModel, 103 links, 102 joints
Links:
- added link l_hand_index_1, mass 1e-5; collision box size=1 1 1; visual box size=1 1 1
- added link l_hand_index_2, mass 1e-5; collision box size=1 1 1; visual box size=1 1 1
- added link l_hand_index_3, mass 1e-5; collision box size=1 1 1; visual box size=1 1 1
- added link l_hand_middle_1, mass 1e-5; collision box size=1 1 1; visual box size=1 1 1
- added link l_hand_middle_2, mass 1e-5; collision box size=1 1 1; visual box size=1 1 1
- added link l_hand_middle_3, mass 1e-5; collision box size=1 1 1; visual box size=1 1 1
- added link l_hand_pinkie_1, mass 1e-5; collision box size=1 1 1; visual box size=1 1 1
- added link l_hand_pinkie_2, mass 1e-5; collision box size=1 1 1; visual box size=1 1 1
- added link l_hand_pinkie_3, mass 1e-5; collision box size=1 1 1; visual box size=1 1 1
- added link l_hand_ring_1, mass 1e-5; collision box size=1 1 1; visual box size=1 1 1
- added link l_hand_ring_2, mass 1e-5; collision box size=1 1 1; visual box size=1 1 1
- added link l_hand_ring_3, mass 1e-5; collision box size=1 1 1; visual box size=1 1 1
- added link l_hand_thumb_1, mass 1e-5; collision box size=1 1 1; visual box size=1 1 1
- added link l_hand_thumb_2, mass 1e-5; collision box size=1 1 1; visual box size=1 1 1
- added link l_hand_thumb_3, mass 1e-5; collision box size=1 1 1; visual box size=1 1 1
- added link r_hand_index_1, mass 1e-5; collision box size=1 1 1; visual box size=1 1 1
- added link r_hand_index_2, mass 1e-5; collision box size=1 1 1; visual box size=1 1 1
- added link r_hand_index_3, mass 1e-5; collision box size=1 1 1; visual box size=1 1 1
- added link r_hand_middle_1, mass 1e-5; collision box size=1 1 1; visual box size=1 1 1
- added link r_hand_middle_2, mass 1e-5; collision box size=1 1 1; visual box size=1 1 1
- added link r_hand_middle_3, mass 1e-5; collision box size=1 1 1; visual box size=1 1 1
- added link r_hand_pinkie_1, mass 1e-5; collision box size=1 1 1; visual box size=1 1 1
- added link r_hand_pinkie_2, mass 1e-5; collision box size=1 1 1; visual box size=1 1 1
- added link r_hand_pinkie_3, mass 1e-5; collision box size=1 1 1; visual box size=1 1 1
- added link r_hand_ring_1, mass 1e-5; collision box size=1 1 1; visual box size=1 1 1
- added link r_hand_ring_2, mass 1e-5; collision box size=1 1 1; visual box size=1 1 1
- added link r_hand_ring_3, mass 1e-5; collision box size=1 1 1; visual box size=1 1 1
- added link r_hand_thumb_1, mass 1e-5; collision box size=1 1 1; visual box size=1 1 1
- added link r_hand_thumb_2, mass 1e-5; collision box size=1 1 1; visual box size=1 1 1
- added link r_hand_thumb_3, mass 1e-5; collision box size=1 1 1; visual box size=1 1 1
Joints:
- added joint l_index_add: type revolute, parent LeftHand, child l_hand_index_1, origin xyz=0.022499999999999958 -0.0015000000000005842 -0.06859999999999963 rpy=0 0 0, axis 0 0 1, limit lower=-0.2617993877991494 upper=0.2617993877991494 effort=30 velocity=1.0
- added joint l_index_dist: type revolute, parent l_hand_index_2, child l_hand_index_3, origin xyz=2.7755575615628914e-17 -0.0015000000000000568 -0.039999999999999925 rpy=0 0 0, axis -1 0 0, limit lower=0 upper=1.7165313193364231 effort=30 velocity=1.0
- added joint l_index_prox: type revolute, parent l_hand_index_1, child l_hand_index_2, origin xyz=0.009192533317427629 1.3877787807814457e-16 -0.030713451316238316 rpy=0 0 0, axis -1 0 0, limit lower=0.10035643198967395 upper=1.710422666954443 effort=30 velocity=1.0
- added joint l_middle_add: type revolute, parent LeftHand, child l_hand_middle_1, origin xyz=0.009599999999999831 -0.0015000000000003344 -0.10299999999999979 rpy=0 0 0, axis 0 0 1, limit lower=-0.2617993877991494 upper=0.2617993877991494 effort=30 velocity=1.0
- added joint l_middle_dist: type revolute, parent l_hand_middle_2, child l_hand_middle_3, origin xyz=-3.122502256758253e-17 -0.0015000000000000568 -0.040000000000000036 rpy=0 0 0, axis -1 0 0, limit lower=0 upper=1.7165313193364231 effort=30 velocity=1.0
- added joint l_middle_prox: type revolute, parent l_hand_middle_1, child l_hand_middle_2, origin xyz=0.009599999999999831 -0.0015000000000003344 -0.10299999999999979 rpy=0 0 0, axis -1 0 0, limit lower=0.10035643198967395 upper=1.710422666954443 effort=30 velocity=1.0
- added joint l_pinkie_add: type revolute, parent LeftHand, child l_hand_pinkie_1, origin xyz=-0.035982322249527375 -0.0023883158589563247 -0.09206560929209864 rpy=0 0 0, axis 0 0 1, limit lower=-0.2617993877991494 upper=0.2617993877991494 effort=30 velocity=1.0
- added joint l_pinkie_dist: type revolute, parent l_hand_pinkie_2, child l_hand_pinkie_3, origin xyz=3.469446951953614e-18 -0.0014999999959518229 -0.03500000000409326 rpy=0 0 0, axis -1 0 0, limit lower=0.04852015320544236 upper=1.7763961126798287 effort=30 velocity=1.0
- added joint l_pinkie_prox: type revolute, parent l_hand_pinkie_1, child l_hand_pinkie_2, origin xyz=-0.035982322249527375 -0.0023883158589563247 -0.09206560929209864 rpy=0 0 0, axis -1 0 0, limit lower=0.10035643198967395 upper=1.710422666954443 effort=30 velocity=1.0
- added joint l_ring_add: type revolute, parent LeftHand, child l_hand_ring_1, origin xyz=-0.015417755558120076 -0.0018498137284708727 -0.09788067183884427 rpy=0 0 0, axis 0 0 1, limit lower=-0.2617993877991494 upper=0.2617993877991494 effort=30 velocity=1.0
- added joint l_ring_dist: type revolute, parent l_hand_ring_2, child l_hand_ring_3, origin xyz=4.336808689942018e-18 -0.0015000000000000568 -0.03999999999999998 rpy=0 0 0, axis -1 0 0, limit lower=0 upper=1.7165313193364231 effort=30 velocity=1.0
- added joint l_ring_prox: type revolute, parent l_hand_ring_1, child l_hand_ring_2, origin xyz=-0.015417755558120076 -0.0018498137284708727 -0.09788067183884427 rpy=0 0 0, axis -1 0 0, limit lower=0.10035643198967395 upper=1.710422666954443 effort=30 velocity=1.0
- added joint l_thumb_add: type revolute, parent LeftHand, child l_hand_thumb_1, origin xyz=0.023374863256390876 -0.003000000000000086 -0.03452383847355481 rpy=0 0 -1.4, axis -1 0 0, limit lower=0 upper=1.7453292519943295 effort=30 velocity=1.0
- added joint l_thumb_dist: type revolute, parent l_hand_thumb_2, child l_hand_thumb_3, origin xyz=-2.7755575615628914e-17 -0.0037106254246525305 -0.03483505790088372 rpy=0 0 0, axis 1 0 0, limit lower=-1.7763961126798287 upper=0 effort=30 velocity=1.0
- added joint l_thumb_prox: type revolute, parent l_hand_thumb_1, child l_hand_thumb_2, origin xyz=-0.03809319745034625 -0.003259193858544507 -0.0036017448037204414 rpy=0 0 0, axis 0 0 1, limit lower=0.0 upper=1.43117 effort=30 velocity=1.0
- added joint r_index_add: type revolute, parent RightHand, child r_hand_index_1, origin xyz=0.022499999999999756 0.0015000000000003344 -0.06859999999999983 rpy=0 0 0, axis 0 0 1, limit lower=-0.2617993877991494 upper=0.2617993877991494 effort=30 velocity=1.0
- added joint r_index_dist: type revolute, parent r_hand_index_2, child r_hand_index_3, origin xyz=4.440892098500626e-16 -0.0014999999999996683 -0.039999999999999925 rpy=0 0 0, axis 1 0 0, limit lower=0 upper=1.7165313193364231 effort=30 velocity=1.0
- added joint r_index_prox: type revolute, parent r_hand_index_1, child r_hand_index_2, origin xyz=-0.00919253331742792 -1.1102230246251565e-16 -0.030713451316238427 rpy=0 0 0, axis 1 0 0, limit lower=0.10035643198967395 upper=1.710422666954443 effort=30 velocity=1.0
- added joint r_middle_add: type revolute, parent RightHand, child r_hand_middle_1, origin xyz=0.009600000000000192 0.0015000000000006675 -0.1029999999999997 rpy=0 0 0, axis 0 0 1, limit lower=-0.2617993877991494 upper=0.2617993877991494 effort=30 velocity=1.0
- added joint r_middle_dist: type revolute, parent r_hand_middle_2, child r_hand_middle_3, origin xyz=3.469446951953614e-16 -0.0014999999953827503 -0.04000000000017301 rpy=0 0 0, axis 1 0 0, limit lower=0 upper=1.7165313193364231 effort=30 velocity=1.0
- added joint r_middle_prox: type revolute, parent r_hand_middle_1, child r_hand_middle_2, origin xyz=0.009600000000000192 0.0015000000000006675 -0.1029999999999997 rpy=0 0 0, axis 1 0 0, limit lower=0.10035643198967395 upper=1.710422666954443 effort=30 velocity=1.0
- added joint r_pinkie_add: type revolute, parent RightHand, child r_hand_pinkie_1, origin xyz=-0.03598268094316618 0.0023777595791096284 -0.0920682813194636 rpy=0 0 0, axis 0 0 1, limit lower=-0.2617993877991494 upper=0.2617993877991494 effort=30 velocity=1.0
- added joint r_pinkie_dist: type revolute, parent r_hand_pinkie_2, child r_hand_pinkie_3, origin xyz=2.8102520310824275e-16 -0.0015141933068321678 -0.03499938883222847 rpy=0 0 0, axis 1 0 0, limit lower=0.04852015320544236 upper=1.7763961126798287 effort=30 velocity=1.0
- added joint r_pinkie_prox: type revolute, parent r_hand_pinkie_1, child r_hand_pinkie_2, origin xyz=-0.03598268094316618 0.0023777595791096284 -0.0920682813194636 rpy=0 0 0, axis 1 0 0, limit lower=0.10035643198967395 upper=1.710422666954443 effort=30 velocity=1.0
- added joint r_ring_add: type revolute, parent RightHand, child r_hand_ring_1, origin xyz=-0.01541775555811984 0.0018498137284709282 -0.09788067183884414 rpy=0 0 0, axis 0 0 1, limit lower=-0.2617993877991494 upper=0.2617993877991494 effort=30 velocity=1.0
- added joint r_ring_dist: type revolute, parent r_hand_ring_2, child r_hand_ring_3, origin xyz=2.8275992658421956e-16 -0.0014999999970887745 -0.04000000000010917 rpy=0 0 0, axis 1 0 0, limit lower=0 upper=1.7165313193364231 effort=30 velocity=1.0
- added joint r_ring_prox: type revolute, parent r_hand_ring_1, child r_hand_ring_2, origin xyz=-0.01541775555811984 0.0018498137284709282 -0.09788067183884414 rpy=0 0 0, axis 1 0 0, limit lower=0.10035643198967395 upper=1.710422666954443 effort=30 velocity=1.0
- added joint r_thumb_add: type revolute, parent RightHand, child r_hand_thumb_1, origin xyz=0.02337486325639067 0.0030000000000002802 -0.034523838473554336 rpy=0.0 0.0 1.4, axis 1 0 0, limit lower=0 upper=1.7453292519943295 effort=30 velocity=1.0
- added joint r_thumb_dist: type revolute, parent r_hand_thumb_2, child r_hand_thumb_3, origin xyz=-8.326672684688674e-17 -0.0037106255282955414 -0.03483505788984376 rpy=0 0 0, axis 1 0 0, limit lower=0 upper=1.7763961126798287 effort=30 velocity=1.0
- added joint r_thumb_prox: type revolute, parent r_hand_thumb_1, child r_hand_thumb_2, origin xyz=0.03807465449956041 0.0034691095803252303 -0.003601744803549689 rpy=0 0 0, axis 0 0 1, limit lower=-1.43117 upper=0.0 effort=30 velocity=1.0
