Commit message: fix fingers prox joint lower limit

File: src/humanmodelgenerator/models/humanModelTemplate/humanModelTemplate.urdf (robot description, URDF)
Before this commit: robot HumanModel, 133 links, 132 joints
Joints:
- joint l_index_prox: limit lower=0.10035643198967395 upper=1.710422666954443 effort=30 velocity=1.0 -> lower=0.0 upper=1.710422666954443 effort=30 velocity=1.0
- joint l_middle_prox: limit lower=0.10035643198967395 upper=1.710422666954443 effort=30 velocity=1.0 -> lower=0.0 upper=1.710422666954443 effort=30 velocity=1.0
- joint l_pinkie_prox: limit lower=0.10035643198967395 upper=1.710422666954443 effort=30 velocity=1.0 -> lower=0.0 upper=1.710422666954443 effort=30 velocity=1.0
- joint l_ring_prox: limit lower=0.10035643198967395 upper=1.710422666954443 effort=30 velocity=1.0 -> lower=0.0 upper=1.710422666954443 effort=30 velocity=1.0
- joint r_index_prox: limit lower=0.10035643198967395 upper=1.710422666954443 effort=30 velocity=1.0 -> lower=0.0 upper=1.710422666954443 effort=30 velocity=1.0
- joint r_middle_prox: limit lower=0.10035643198967395 upper=1.710422666954443 effort=30 velocity=1.0 -> lower=0.0 upper=1.710422666954443 effort=30 velocity=1.0
- joint r_pinkie_prox: limit lower=0.10035643198967395 upper=1.710422666954443 effort=30 velocity=1.0 -> lower=0.0 upper=1.710422666954443 effort=30 velocity=1.0
- joint r_ring_prox: limit lower=0.10035643198967395 upper=1.710422666954443 effort=30 velocity=1.0 -> lower=0.0 upper=1.710422666954443 effort=30 velocity=1.0
